File: hw/LED_PCB/led_pcb.brd (EAGLE design)
At the start: 110 x 55 mm, 99 parts, among them J1 INPUT, J2 OUTPUT, J3 POWER, U1 WS2813, U10 WS2813, U11 WS2813, U12 WS2813, U13 WS2813, U14 WS2813, U15 WS2813, U16 WS2813, U17 WS2813, U18 WS2813, U19 WS2813, U2 WS2813, U20 WS2813, U21 WS2813, U22 WS2813, U23 WS2813, U24 WS2813, U25 WS2813, U26 WS2813, U27 WS2813, U28 WS2813, U29 WS2813, U3 WS2813, U30 WS2813, U31 WS2813, U32 WS2813, U4 WS2813, U5 WS2813, U6 WS2813, U7 WS2813, U8 WS2813, U9 WS2813

Commit message: Final touches on LED pcb
Parts:
- J1, J2, J3: device SparkFun-Connectors:2X5-SHROUDED_SMD -> kala_lib:2X5-SHROUDED_SMD
- moved C28 1.16 mm to (52.0, 14.6)
- moved C8 0.90 mm to (106.9, 43.7)
- moved C17 0.85 mm to (9.20, 16.1)
- moved C29 0.81 mm to (67.8, 3.74)
- moved R16 0.53 mm to (96.9, 39.9)
- moved R17 0.45 mm to (13.4, 19.1)
- moved C9 0.30 mm to (13.9, 28.8)
Routing:
- net N$18: track 11.2 -> 13.4 mm
- net N$15: track 9.14 -> 10.9 mm
- net DO15: track 128.9 -> 130.5 mm
- net N$53: track 16.4 -> 17.6 mm
- net N$55: track 8.84 -> 10.0 mm
- net N$36: track 20.3 -> 20.8 mm
