File: hw/Hat_PCB/Hat_PCB.sch (KiCad schematic (older format))
At the start: 15 parts, among them J3 40HAT, J9 CONN_01X02, Q1 DMG2305UX, Q2 DMMT5401, U2 CAT24C32

Commit message: Add schematic symbols for most components
Parts:
- added U?: ATtiny88-MU, Package_DFN_QFN:QFN-32-1EP_5x5mm_P0.5mm_EP3.1x3.1mm, symbol MCU_Microchip_ATtiny:ATtiny88-MU
- added U?: BME680, Package_LGA:Bosch_LGA-8_3x3mm_P0.8mm_ClockwisePinNumbering, symbol Sensor:BME680
- added U?: MPR121QR2, QFN40P300X300X60-20N, symbol MPR121QR2:MPR121QR2
- added U?: TPA2016D2RTJR, QFN50P400X400X80-21N, symbol TPA2016D2RTJR:TPA2016D2RTJR
- added U?: TSL2591, Package_DFN_QFN:DFN-6_1.3x1.2mm_P0.4mm, symbol tsl2591:TSL2591
Changed lines of the file:
@@
 Wire Wire Line
 	1050 6100 1150 6100
+$Comp
+L MCU_Microchip_ATtiny:ATtiny88-MU U?
+U 1 1 5C3B6615
+P 5400 9200
+F 0 "U?" H 4870 9154 50  0000 R CNN
+F 1 "ATtiny88-MU" H 4870 9245 50  0000 R CNN
+F 2 "Package_DFN_QFN:QFN-32-1EP_5x5mm_P0.5mm_EP3.1x3.1mm" H 5400 9200 50  0001 C CIN
+F 3 "http://ww1.microchip.com/downloads/en/DeviceDoc/doc8008.pdf" H 5400 9200 50  0001 C CNN
+	1    5400 9200
+	1    0    0    -1
+$EndComp
+$Comp
+L Sensor:BME680 U?
+U 1 1 5C3BDBAD
+P 6200 5250
+F 0 "U?" H 5770 5296 50  0000 R CNN
+F 1 "BME680" H 5770 5205 50  0000 R CNN
+F 2 "Package_LGA:Bosch_LGA-8_3x3mm_P0.8mm_ClockwisePinNumbering" H 6200 5050 50  0001 C CNN
+F 3 "https://ae-bst.resource.bosch.com/media/_tech/media/datasheets/BST-BME680-DS001-00.pdf" H 6200 5050 50  0001 C CNN
+	1    6200 5250
+	1    0    0    -1
+$EndComp
+$Comp
+L MPR121QR2:MPR121QR2 U?
+U 1 1 5C3BF345
+P 11850 3600
+F 0 "U?" H 11850 4370 50  0000 C CNN
+F 1 "MPR121QR2" H 11850 4279 50  0000 C CNN
+F 2 "QFN40P300X300X60-20N" H 11850 3600 50  0001 L BNN
+F 3 "Unavailable" H 11850 3600 50  0001 L BNN
+F 4 "NXP USA" H 11850 3600 50  0001 L BNN "Field4"
+F 5 "Capacitive Touch Screen 12Keys 20-Pin QFN Tape and Reel" H 11850 3600 50  0001 L BNN "Field5"
+F 6 "None" H 11850 3600 50  0001 L BNN "Field6"
+F 7 "QFN-20 Freescale Semiconductor" H 11850 3600 50  0001 L BNN "Field7"
+F 8 "MPR121QR2" H 11850 3600 50  0001 L BNN "Field8"
+	1    11850 3600
+	1    0    0    -1
+$EndComp
+$Comp
+L TPA2016D2RTJR:TPA2016D2RTJR U?
+U 1 1 5C3BF5FA
+P 12000 7100
+F 0 "U?" H 12000 8370 50  0000 C CNN
+F 1 "TPA2016D2RTJR" H 12000 8279 50  0000 C CNN
+F 2 "QFN50P400X400X80-21N" H 12000 7100 50  0001 L BNN
+F 3 "Unavailable" H 12000 7100 50  0001 L BNN
+F 4 "Texas Instruments" H 12000 7100 50  0001 L BNN "Field4"
+F 5 "2.8-W/Ch Stereo Class-D Audio Amplifier with SmartGainTM AGC/DRC _TPA2016_ 20-QFN -40 to 85" H 12000 7100 50  0001 L BNN "Field5"
+F 6 "None" H 12000 7100 50  0001 L BNN "Field6"
+F 7 "QFN-20 Texas Instruments" H 12000 7100 50  0001 L BNN "Field7"
+F 8 "TPA2016D2RTJR" H 12000 7100 50  0001 L BNN "Field8"
+	1    12000 7100
+	1    0    0    -1
+$EndComp
+$Comp
+L tsl2591:TSL2591 U?
+U 1 1 5C3C1FDB
+P 8550 10100
+F 0 "U?" H 8675 10225 50  0000 C CNN
+F 1 "TSL2591" H 8675 10134 50  0000 C CNN
+F 2 "Package_DFN_QFN:DFN-6_1.3x1.2mm_P0.4mm" H 8550 10150 50  0001 C CNN
+F 3 "" H 8550 10150 50  0001 C CNN
+	1    8550 10100
+	1    0    0    -1
+$EndComp
 $EndSCHEMATC

Commit message: Schematic mostly done, started prelim layout
Parts:
- added C1, C12, C13, C4, C5: 10uF, Capacitor_SMD:C_0603_1608Metric_Pad1.05x0.95mm_HandSolder, symbol Device:C
- added C10, C11, C2, C3, C6, C7, C8, C9: 0.1uF, Capacitor_SMD:C_0603_1608Metric_Pad1.05x0.95mm_HandSolder, symbol Device:C
- added J1: ATTINY_ICSP, Connector_PinHeader_2.54mm:PinHeader_1x06_P2.54mm_Vertical, symbol Connector_Generic:Conn_01x06
- added J2: I2C, Connector_PinHeader_2.54mm:PinHeader_1x02_P2.54mm_Vertical, symbol Connector_Generic:Conn_01x02
- added J4: RPi_Power, Connector_PinHeader_2.54mm:PinHeader_1x02_P2.54mm_Vertical, symbol Connector_Generic:Conn_01x02
- added J5: AUD_IN, Connector_PinHeader_2.54mm:PinHeader_1x04_P2.54mm_Vertical, symbol Connector_Generic:Conn_01x04
- added J6: OUT_SPK_L, Connector_PinHeader_2.54mm:PinHeader_1x02_P2.54mm_Vertical, symbol Connector_Generic:Conn_01x02
- added J7: OUT_SPK_R, Connector_PinHeader_2.54mm:PinHeader_1x02_P2.54mm_Vertical, symbol Connector_Generic:Conn_01x02
- added J8: CAP_TOUCH, Connector_PinHeader_2.54mm:PinHeader_1x12_P2.54mm_Vertical, symbol Connector_Generic:Conn_01x12
- added MK1, MK2: SPH0645LM4H-B, MIC_SPH0645LM4H-B, symbol SPH0645LM4H-B:SPH0645LM4H-B
- added R1, R2, R3, R7: 33R, Resistor_SMD:R_0603_1608Metric_Pad1.05x0.95mm_HandSolder, symbol Device:R
- added R10, R12, R18, R9: 10K, Resistor_SMD:R_0603_1608Metric_Pad1.05x0.95mm_HandSolder, symbol Device:R
- added R13: 68R, Resistor_SMD:R_0603_1608Metric_Pad1.05x0.95mm_HandSolder, symbol Device:R
- added R14, R15, R16: 0R, Resistor_SMD:R_0603_1608Metric_Pad1.05x0.95mm_HandSolder, symbol Device:R
- added R17: 75K, Resistor_SMD:R_0603_1608Metric_Pad1.05x0.95mm_HandSolder, symbol Device:R
- added R4, R5: 3.9K, Resistor_SMD:R_0603_1608Metric_Pad1.05x0.95mm_HandSolder, symbol Device:R
- added U7: NCP1117-3.3_SOT223, Package_TO_SOT_SMD:SOT-223-3_TabPin2, symbol Regulator_Linear:NCP1117-3.3_SOT223
- J9: value CONN_01X02 -> EE_WP
- R11, R23, R24, R29: footprint Resistor_SMD:R_0603_1608Metric_Pad0.84x1.00mm_HandSolder -> Resistor_SMD:R_0603_1608Metric_Pad1.05x0.95mm_HandSolder
- R6: value 3.9K -> 33R; footprint Resistor_SMD:R_0603_1608Metric_Pad0.84x1.00mm_HandSolder -> Resistor_SMD:R_0603_1608Metric_Pad1.05x0.95mm_HandSolder
- R8: value 3.9K -> 10K; footprint Resistor_SMD:R_0603_1608Metric_Pad0.84x1.00mm_HandSolder -> Resistor_SMD:R_0603_1608Metric_Pad1.05x0.95mm_HandSolder
- U1: renamed from U?; value ATtiny88-MU -> ATtiny87-MU; symbol MCU_Microchip_ATtiny:ATtiny88-MU -> MCU_Microchip_ATtiny:ATtiny87-MU
- U4: renamed from U?; symbol tsl2591:TSL2591 -> Hat_PCB-rescue:TSL2591-tsl2591
- U5: renamed from U?; footprint QFN40P300X300X60-20N -> Package_DFN_QFN:QFN-20-1EP_3x3mm_P0.45mm_EP1.6x1.6mm; symbol MPR121QR2:MPR121QR2 -> Hat_PCB-rescue:MPR121QR2-MPR121QR2
- U6: renamed from U?; footprint QFN50P400X400X80-21N -> Package_DFN_QFN:QFN-20-1EP_4x4mm_P0.5mm_EP2.5x2.5mm; symbol TPA2016D2RTJR:TPA2016D2RTJR -> Hat_PCB-rescue:TPA2016D2RTJR-TPA2016D2RTJR
- gave numbers to parts that had none: 1
Connections:
- net labels added: +3.3V, +5V, ALS_INT, AUD_IN_L+, AUD_IN_L-, AUD_IN_R+, AUD_IN_R-, AUD_SDN, CAP_IRQ, GPIO_PB1, GPIO_PB3, GPIO_PB4, GPIO_PB5, ID_SC, ID_SD, LED_DATA, MCU_AREF, MCU_INT, MCU_RXD, MCU_TXD, MIC_CLK, MIC_DO, MIC_WS, PROG_CLK, PROG_MISO, PROG_MOSI, PROG_RST_N, PROG_SCK, PSUP_5V, Pi_3V3, SCL, SDA, SPI_CS_N
- net labels removed: ID_SC_EEPROM, ID_SC_EEPROM_pu, ID_SD_EEPROM, ID_SD_EEPROM_pu, P3V3, P3V3_HAT, P5V, P5V_HAT
- wire segments 66 -> 302
Other:
- note added: "3.3V LDO Regulator"
- note added: "ADDR: I2C Address Bit\nVSS: 0x5A\nVDD: 0x5B\nSDA: 0x5C\nSCL: 0x5D\n"
- note added: "Ambient Light Sensor"
- note added: "Audio Amplifier"
- note added: "Cap Touch"
- note added: "Gas, Pressure, Temp, Humidity Sense"
- note added: "I2C Address: 0x5A"
- note added: "I2C Address: 0x66"
- note added: "I2C Address: 0x77"
- note added: "I2C Addresses: \n0xB0 (Writing)\n0xB1 (Reading)"
- note added: "LED Driver"
- note added: "LEFT CHANNEL MIC"
- note added: "MEMS I2S Stereo Microphones"
- note added: "RIGHT CHANNEL MIC"
- note added: "SDO: I2C Address Bit\nGND: 0 (0x76)\nVCC: 1 (0x77)\n"
- note removed: "EEPROM WRITE ENABLE"
- note removed: "Pullup Resistors"
- note removed: "The HAT spec requires this EEPROM with system information\nto be in place in order to be called a HAT. It should be set up as write\nprotected (WP pin held high), so it may be desirable to either put a \njumper as shown to enable writing, or to hook up a spare IO pin to do so."
- note removed: "These are just pullup resistors for the I2C bus on the EEPROM.\nThe resistor values are per the HAT spec."
- note removed: "This is based on the official Raspberry Pi spec to be able to call an extension board a HAT.\nhttps://github.com/raspberrypi/hats/blob/master/designguide.md"
- note removed: "This is the recommended 5V rail protection for \na HAT with power going to the Pi.\nSee https://github.com/raspberrypi/hats/blob/master/designguide.md#back-powering-the-pi-via-the-j8-gpio-header"
- moved on the sheet: J3, J9, Q1, Q2A, Q2B, R11, R23, R24, R29, U2, U3

Commit message: Added RTC, changed layout a bit
Parts:
- removed J1: ATTINY_ICSP, Connector_PinHeader_2.54mm:PinHeader_1x06_P2.54mm_Vertical, symbol Connector_Generic:Conn_01x06
- added BT1: Battery_Cell, Battery:BatteryHolder_Keystone_3000_1x12mm, symbol Device:Battery_Cell
- added D1: BAV99, SOT23-3, symbol BAV99:BAV99
- added J10: AudioJack3, Connector_Audio:Jack_3.5mm_CUI_SJ1-3533NG_Horizontal, symbol Connector:AudioJack3
- added J11: AudioJack3_Ground, Connector_Audio:Jack_3.5mm_CUI_SJ1-3533NG_Horizontal, symbol Connector:AudioJack3
- added J3: AVR-ISP-6, Connector_PinHeader_2.54mm:PinHeader_2x03_P2.54mm_Vertical, symbol Connector:AVR-ISP-6
- added U6: DS3231M, Package_SO:SOIC-16W_7.5x10.3mm_P1.27mm, symbol Timer_RTC:DS3231M
- U1: renamed from U2; footprint Package_SOIC:SOIC-8_3.9x4.9mm_P1.27mm -> Package_SO:SOIC-8_3.9x4.9mm_P1.27mm
- renumbered H3 to H2, H2 to H3, J9 to J1, J3 to J2, J2 to J4, J4 to J5, J5 to J6, J6 to J7, J7 to J8, J8 to J9, Q2 to Q1, Q1 to Q2, R23 to R10, R8 to R11, R24 to R12, R10 to R13, R9 to R14, R12 to R15, R13 to R16, R14 to R17, R15 to R18, R16 to R19, R17 to R20, R18 to R21, R11 to R4, R29 to R5, R4 to R6, R5 to R7, R6 to R8, R7 to R9, U1 to U2, U7 to U3, U3 to U5, U6 to U7, U5 to U8
Connections:
- net +3V3: now also D1.2 (C2), J3.2 (VCC), U6.2 (VCC)
- net AUD_IN_L+: now also J10.T
- net AUD_IN_R+: now also J10.R
- net GND: now also BT1.2 (-), D1.1 (A1), J10.S, J11.S, J3.6 (GND), U6.10 (GND), U6.11 (GND), U6.12 (GND), U6.13 (GND), U6.5 (GND), U6.6 (GND), U6.7 (GND), U6.8 (GND), U6.9 (GND)
- net PROG_MISO: now also J3.1 (MISO)
- net PROG_MOSI: now also J3.4 (MOSI)
- net PROG_RST_N: now also D1.3 (COM), J3.5 (~RST)
- net PROG_SCK: now also J3.3 (SCK)
- net SCL: now also U6.16 (SCL)
- net SDA: now also U6.15 (SDA)
- net AUD_O_R+: now reaches J8.1 (Pin_1), U7.10 (OUTR+)
- net AUD_O_R+: now also J11.R
- net AUD_O_L+: now reaches J7.1 (Pin_1), U7.6 (OUTL+)
- net AUD_O_L+: now also J11.T
- net AUD_O_L-: now reaches J7.2 (Pin_2), U7.7 (OUTL-)
- net AUD_O_R-: now reaches J8.2 (Pin_2), U7.9 (OUTR-)
- new net: BT1.1 (+), U6.14 (VBAT)
- new net RTC_32KHZ: U6.1 (32KHZ)
- new net RTC_INT: U6.3 (~INT~/SQW)
- new net RTC_RST: U6.4 (~RST)
Other:
- note added: "I2C Address: 0x29"
- note added: "I2C Address: 0x68"
- note added: "Real Time Clock"
- note added: "To do:\n- Power / indicator LEDs\n- I2C pull ups\n- Better connectors\n- Double check reference schematics for possible missing parts\n- Placement for passives"
- moved on the sheet: C8, J7, J8, R13, U4

Commit message: Added pull ups, LEDs, & swapped out cap touch IC
Parts:
- removed C10: 0.1uF, Capacitor_SMD:C_0603_1608Metric_Pad1.05x0.95mm_HandSolder, symbol Device:C
- removed R20: 75K, Resistor_SMD:R_0603_1608Metric_Pad1.05x0.95mm_HandSolder, symbol Device:R
- removed R5: 10K, Resistor_SMD:R_0603_1608Metric_Pad1.05x0.95mm_HandSolder, symbol Device:R
- removed U8: MPR121QR2, Package_DFN_QFN:QFN-20-1EP_3x3mm_P0.45mm_EP1.6x1.6mm, symbol Hat_PCB-rescue:MPR121QR2-MPR121QR2
- added D?: 5V_LED, symbol Device:LED_ALT
- added D?: 3V3_LED, symbol Device:LED_ALT
- added D?: GPIO_LED, symbol Device:LED_ALT
- added J?: I2C, Connector_PinHeader_2.54mm:PinHeader_1x02_P2.54mm_Vertical, symbol Connector_Generic:Conn_01x02
- added R? (x3): 330R, Resistor_SMD:R_0603_1608Metric_Pad1.05x0.95mm_HandSolder, symbol Device:R
- added R? (x2): 3.9K, Resistor_SMD:R_0603_1608Metric_Pad1.05x0.95mm_HandSolder, symbol Device:R
- added R?: 10K, Resistor_SMD:R_0603_1608Metric_Pad1.05x0.95mm_HandSolder, symbol Device:R
- added R? (x2): 33R, Resistor_SMD:R_0603_1608Metric_Pad1.05x0.95mm_HandSolder, symbol Device:R
- added R?: 47K, Resistor_SMD:R_0603_1608Metric_Pad1.05x0.95mm_HandSolder, symbol Device:R
- added U?: AT42QT2120-MMH, QFN45P300X300X85-21N, symbol AT42QT2120-MMH:AT42QT2120-MMH
- J4: value I2C -> ID_I2C
Connections:
- net +3V3: now also D?.2 (A), R?.1, R?.1, R?.1, R?.2, U?.9 (VDD)
- net +5V: now also D?.2 (A)
- net GND: now also R?.1, R?.1, R?.1, U?.10 (MODE), U?.21 (EP), U?.8 (VSS)
- net GPIO_PB1: now also D?.2 (A)
- net MCU_RXD: now also R?.2
- net MCU_TXD: now also R?.2
- net SCL: now also J?.2 (Pin_2), R?.2, U?.11 (SDA)
- net SDA: now also J?.1 (Pin_1), R?.2, U?.14 (SCL)
- net at J2.10 (BCM15): now also R?.1
- net at J2.8 (BCM14): now also R?.1
- net at J1.2 (Pin_2), R4.1, U1.7 (WP): now also R?.1
- net at J9.3 (Pin_3): now also U?.5 (KEY2)
- net at J9.4 (Pin_4): now also U?.4 (KEY3)
- net at J9.5 (Pin_5): now also U?.3 (KEY4)
- net at J9.6 (Pin_6): now also U?.2 (KEY5)
- net at J9.7 (Pin_7): now also U?.1 (KEY6)
- net at J9.8 (Pin_8): now also U?.20 (KEY7)
- net at J9.9 (Pin_9): now also U?.19 (KEY8)
- net at J9.10 (Pin_10): now also U?.18 (KEY9)
- net at J9.11 (Pin_11): now also U?.17 (KEY10)
- net at J9.12 (Pin_12): now also U?.16 (KEY11)
- net at J9.1 (Pin_1): now also U?.7 (KEY0)
- net at J9.2 (Pin_2): now also U?.6 (KEY1)
- net CAP_IRQ: no longer names the net of R21.2
- net CAP_IRQ: now also U?.12 (~RST)
- new net: D?.1 (K), R?.2 (x3)
- new net: R?.2, U?.15 (~INT)
Other:
- note added: "ATTINY LED Driver"
- note added: "I2C Address: 0x1C"
- note added: "I2C Pull Ups"
- note added: "Indicator LEDs"
- note added: "To do:\n- Better connectors\n- Double check reference schematics for possible missing parts\n- Placement for passives"
- note removed: "ADDR: I2C Address Bit\nVSS: 0x5A\nVDD: 0x5B\nSDA: 0x5C\nSCL: 0x5D\n"
- note removed: "I2C Address: 0x5A"
- note removed: "LED Driver"
- note removed: "To do:\n- Power / indicator LEDs\n- I2C pull ups\n- Better connectors\n- Double check reference schematics for possible missing parts\n- Placement for passives"
- moved on the sheet: C1, C2, C3, C4, C5, C8, C9, D1, J3, J9, R11, R13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
