File: hw/Main_LED_PCB_v2/main_led_pcb/_autosave-main_led_pcb.kicad_pcb (KiCad board)
At the start: 2 copper layers, 220 x 220 mm, 539 parts, among them J1 PWR_IN, J2 AVR-ISP-6, J3 UART, J4 I2C, J5 PA, J6 PB, U1 ATtiny87-MU, U2 NCP1117-3.3_SOT223

Commit message: Add all files, sort out later
Parts:
- moved R177 344.8 mm to (7.00, 157.6)
- moved R241 342.4 mm to (7.00, 212.0)
- moved R242 341.1 mm to (20.5, 212.0)
- moved R245 336.7 mm to (61.1, 212.0)
- moved R225 335.8 mm to (7.00, 198.4)
- moved R179 335.0 mm to (34.1, 157.6)
- moved R226 334.3 mm to (20.5, 198.4)
- moved R209 329.4 mm to (7.00, 184.8)
- moved R161 327.9 mm to (7.00, 144.0)
- moved R210 327.7 mm to (20.5, 184.8)
- moved R129 321.5 mm to (7.00, 116.8)
- moved R246 316.3 mm to (74.7, 212.0)
- moved R231 316.0 mm to (88.2, 198.4)
- moved R213 314.4 mm to (61.1, 184.8)
- moved R145 314.4 mm to (7.00, 130.4)
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Connections:
- D1 pad 2: Net-(D1-Pad2) -> +5V
- D1 pad 5: Net-(D1-Pad5) -> GND
- D10 pad 2: Net-(D10-Pad2) -> +5V
- D10 pad 5: Net-(D10-Pad5) -> GND
- D100 pad 2: Net-(D100-Pad2) -> +5V
- D100 pad 5: Net-(D100-Pad5) -> GND
- D101 pad 2: Net-(D101-Pad2) -> +5V
- D101 pad 5: Net-(D101-Pad5) -> GND
- D102 pad 2: Net-(D102-Pad2) -> +5V
- D102 pad 5: Net-(D102-Pad5) -> GND
- D103 pad 2: Net-(D103-Pad2) -> +5V
- D103 pad 5: Net-(D103-Pad5) -> GND
- D104 pad 2: Net-(D104-Pad2) -> +5V
- D104 pad 5: Net-(D104-Pad5) -> GND
- D105 pad 2: Net-(D105-Pad2) -> +5V
- D105 pad 5: Net-(D105-Pad5) -> GND
- D106 pad 2: Net-(D10-Pad2) -> +5V
- D106 pad 5: Net-(D10-Pad5) -> GND
- D107 pad 2: Net-(D107-Pad2) -> +5V
- D107 pad 5: Net-(D107-Pad5) -> GND
- D108 pad 2: Net-(D108-Pad2) -> +5V
- D108 pad 5: Net-(D108-Pad5) -> GND
- D109 pad 2: Net-(D109-Pad2) -> +5V
- D109 pad 5: Net-(D109-Pad5) -> GND
- D11 pad 2: Net-(D107-Pad2) -> +5V
- D11 pad 5: Net-(D107-Pad5) -> GND
- D110 pad 2: Net-(D110-Pad2) -> +5V
- D110 pad 5: Net-(D110-Pad5) -> GND
- D111 pad 2: Net-(D111-Pad2) -> +5V
- D111 pad 5: Net-(D111-Pad5) -> GND
- D112 pad 2: Net-(D112-Pad2) -> +5V
- D112 pad 5: Net-(D112-Pad5) -> GND
- D113 pad 2: Net-(D1-Pad2) -> +5V
- D113 pad 5: Net-(D1-Pad5) -> GND
- D114 pad 2: Net-(D114-Pad2) -> +5V
- D114 pad 5: Net-(D114-Pad5) -> GND
- D115 pad 2: Net-(D115-Pad2) -> +5V
- D115 pad 5: Net-(D115-Pad5) -> GND
- D116 pad 2: Net-(D100-Pad2) -> +5V
- D116 pad 5: Net-(D100-Pad5) -> GND
- D117 pad 2: Net-(D101-Pad2) -> +5V
- D117 pad 5: Net-(D101-Pad5) -> GND
- D118 pad 2: Net-(D102-Pad2) -> +5V
- D118 pad 5: Net-(D102-Pad5) -> GND
- D119 pad 2: Net-(D103-Pad2) -> +5V
- D119 pad 5: Net-(D103-Pad5) -> GND
- D12 pad 2: Net-(D108-Pad2) -> +5V
- D12 pad 5: Net-(D108-Pad5) -> GND
- D120 pad 2: Net-(D104-Pad2) -> +5V
- D120 pad 5: Net-(D104-Pad5) -> GND
- D121 pad 2: Net-(D105-Pad2) -> +5V
- D121 pad 5: Net-(D105-Pad5) -> GND
- D122 pad 2: Net-(D10-Pad2) -> +5V
- D122 pad 5: Net-(D10-Pad5) -> GND
- D123 pad 2: Net-(D107-Pad2) -> +5V
- D123 pad 5: Net-(D107-Pad5) -> GND
- D124 pad 2: Net-(D108-Pad2) -> +5V
- D124 pad 5: Net-(D108-Pad5) -> GND
- D125 pad 2: Net-(D109-Pad2) -> +5V
- D125 pad 5: Net-(D109-Pad5) -> GND
- D126 pad 2: Net-(D110-Pad2) -> +5V
- D126 pad 5: Net-(D110-Pad5) -> GND
- D127 pad 2: Net-(D111-Pad2) -> +5V
- D127 pad 5: Net-(D111-Pad5) -> GND
- D128 pad 2: Net-(D112-Pad2) -> +5V
- D128 pad 5: Net-(D112-Pad5) -> GND
- D129 pad 2: Net-(D1-Pad2) -> +5V
- D129 pad 5: Net-(D1-Pad5) -> GND
- D13 pad 2: Net-(D109-Pad2) -> +5V
- D13 pad 5: Net-(D109-Pad5) -> GND
- D130 pad 2: Net-(D114-Pad2) -> +5V
- D130 pad 5: Net-(D114-Pad5) -> GND
- D131 pad 2: Net-(D115-Pad2) -> +5V
- D131 pad 5: Net-(D115-Pad5) -> GND
- D132 pad 2: Net-(D100-Pad2) -> +5V
- D132 pad 5: Net-(D100-Pad5) -> GND
- D133 pad 2: Net-(D101-Pad2) -> +5V
- D133 pad 5: Net-(D101-Pad5) -> GND
- D134 pad 2: Net-(D102-Pad2) -> +5V
- D134 pad 5: Net-(D102-Pad5) -> GND
- D135 pad 2: Net-(D103-Pad2) -> +5V
- D135 pad 5: Net-(D103-Pad5) -> GND
- D136 pad 2: Net-(D104-Pad2) -> +5V
- D136 pad 5: Net-(D104-Pad5) -> GND
- D137 pad 2: Net-(D105-Pad2) -> +5V
- D137 pad 5: Net-(D105-Pad5) -> GND
- D138 pad 2: Net-(D10-Pad2) -> +5V
- D138 pad 5: Net-(D10-Pad5) -> GND
- D139 pad 2: Net-(D107-Pad2) -> +5V
- D139 pad 5: Net-(D107-Pad5) -> GND
- D14 pad 2: Net-(D110-Pad2) -> +5V
- D14 pad 5: Net-(D110-Pad5) -> GND
- D140 pad 2: Net-(D108-Pad2) -> +5V
- D140 pad 5: Net-(D108-Pad5) -> GND
- D141 pad 2: Net-(D109-Pad2) -> +5V
- D141 pad 5: Net-(D109-Pad5) -> GND
- D142 pad 2: Net-(D110-Pad2) -> +5V
- D142 pad 5: Net-(D110-Pad5) -> GND
- D143 pad 2: Net-(D111-Pad2) -> +5V
- D143 pad 5: Net-(D111-Pad5) -> GND
- D144 pad 2: Net-(D112-Pad2) -> +5V
- D144 pad 5: Net-(D112-Pad5) -> GND
- D145 pad 2: Net-(D1-Pad2) -> +5V
- D145 pad 5: Net-(D1-Pad5) -> GND
- D146 pad 2: Net-(D114-Pad2) -> +5V
- D146 pad 5: Net-(D114-Pad5) -> GND
- D147 pad 2: Net-(D115-Pad2) -> +5V
- D147 pad 5: Net-(D115-Pad5) -> GND
- D148 pad 2: Net-(D100-Pad2) -> +5V
- D148 pad 5: Net-(D100-Pad5) -> GND
- D149 pad 2: Net-(D101-Pad2) -> +5V
- D149 pad 5: Net-(D101-Pad5) -> GND
- D15 pad 2: Net-(D111-Pad2) -> +5V
- D15 pad 5: Net-(D111-Pad5) -> GND
- D150 pad 2: Net-(D102-Pad2) -> +5V
- D150 pad 5: Net-(D102-Pad5) -> GND
- D151 pad 2: Net-(D103-Pad2) -> +5V
- D151 pad 5: Net-(D103-Pad5) -> GND
- D152 pad 2: Net-(D104-Pad2) -> +5V
- D152 pad 5: Net-(D104-Pad5) -> GND
- D153 pad 2: Net-(D105-Pad2) -> +5V
- D153 pad 5: Net-(D105-Pad5) -> GND
- D154 pad 2: Net-(D10-Pad2) -> +5V
- D154 pad 5: Net-(D10-Pad5) -> GND
- D155 pad 2: Net-(D107-Pad2) -> +5V
- D155 pad 5: Net-(D107-Pad5) -> GND
- D156 pad 2: Net-(D108-Pad2) -> +5V
- D156 pad 5: Net-(D108-Pad5) -> GND
- D157 pad 2: Net-(D109-Pad2) -> +5V
- D157 pad 5: Net-(D109-Pad5) -> GND
- D158 pad 2: Net-(D110-Pad2) -> +5V
- D158 pad 5: Net-(D110-Pad5) -> GND
- D159 pad 2: Net-(D111-Pad2) -> +5V
- D159 pad 5: Net-(D111-Pad5) -> GND
- D16 pad 2: Net-(D112-Pad2) -> +5V
- D16 pad 5: Net-(D112-Pad5) -> GND
- D160 pad 2: Net-(D112-Pad2) -> +5V
- D160 pad 5: Net-(D112-Pad5) -> GND
- D161 pad 2: Net-(D1-Pad2) -> +5V
- D161 pad 5: Net-(D1-Pad5) -> GND
- D162 pad 2: Net-(D114-Pad2) -> +5V
- D162 pad 5: Net-(D114-Pad5) -> GND
- D163 pad 2: Net-(D115-Pad2) -> +5V
- D163 pad 5: Net-(D115-Pad5) -> GND
- D164 pad 2: Net-(D100-Pad2) -> +5V
- D164 pad 5: Net-(D100-Pad5) -> GND
- D165 pad 2: Net-(D101-Pad2) -> +5V
- D165 pad 5: Net-(D101-Pad5) -> GND
- D166 pad 2: Net-(D102-Pad2) -> +5V
- D166 pad 5: Net-(D102-Pad5) -> GND
- D167 pad 2: Net-(D103-Pad2) -> +5V
- D167 pad 5: Net-(D103-Pad5) -> GND
- D168 pad 2: Net-(D104-Pad2) -> +5V
- D168 pad 5: Net-(D104-Pad5) -> GND
- D169 pad 2: Net-(D105-Pad2) -> +5V
- D169 pad 5: Net-(D105-Pad5) -> GND
- D17 pad 2: Net-(D1-Pad2) -> +5V
- D17 pad 5: Net-(D1-Pad5) -> GND
- D170 pad 2: Net-(D10-Pad2) -> +5V
- D170 pad 5: Net-(D10-Pad5) -> GND
- D171 pad 2: Net-(D107-Pad2) -> +5V
- D171 pad 5: Net-(D107-Pad5) -> GND
- D172 pad 2: Net-(D108-Pad2) -> +5V
- D172 pad 5: Net-(D108-Pad5) -> GND
- D173 pad 2: Net-(D109-Pad2) -> +5V
- D173 pad 5: Net-(D109-Pad5) -> GND
- D174 pad 2: Net-(D110-Pad2) -> +5V
- D174 pad 5: Net-(D110-Pad5) -> GND
- D175 pad 2: Net-(D111-Pad2) -> +5V
- D175 pad 5: Net-(D111-Pad5) -> GND
- D176 pad 2: Net-(D112-Pad2) -> +5V
- D176 pad 5: Net-(D112-Pad5) -> GND
- D177 pad 2: Net-(D1-Pad2) -> +5V
- D177 pad 5: Net-(D1-Pad5) -> GND
- D178 pad 2: Net-(D114-Pad2) -> +5V
- D178 pad 5: Net-(D114-Pad5) -> GND
- D179 pad 2: Net-(D115-Pad2) -> +5V
- D179 pad 5: Net-(D115-Pad5) -> GND
- D18 pad 2: Net-(D114-Pad2) -> +5V
- D18 pad 5: Net-(D114-Pad5) -> GND
- D180 pad 2: Net-(D100-Pad2) -> +5V
- D180 pad 5: Net-(D100-Pad5) -> GND
- D181 pad 2: Net-(D101-Pad2) -> +5V
- D181 pad 5: Net-(D101-Pad5) -> GND
- D182 pad 2: Net-(D102-Pad2) -> +5V
- D182 pad 5: Net-(D102-Pad5) -> GND
- D183 pad 2: Net-(D103-Pad2) -> +5V
- D183 pad 5: Net-(D103-Pad5) -> GND
- D184 pad 2: Net-(D104-Pad2) -> +5V
- D184 pad 5: Net-(D104-Pad5) -> GND
- D185 pad 2: Net-(D105-Pad2) -> +5V
- D185 pad 5: Net-(D105-Pad5) -> GND
- D186 pad 2: Net-(D10-Pad2) -> +5V
- D186 pad 5: Net-(D10-Pad5) -> GND
- D187 pad 2: Net-(D107-Pad2) -> +5V
- D187 pad 5: Net-(D107-Pad5) -> GND
- D188 pad 2: Net-(D108-Pad2) -> +5V
- D188 pad 5: Net-(D108-Pad5) -> GND
- D189 pad 2: Net-(D109-Pad2) -> +5V
- D189 pad 5: Net-(D109-Pad5) -> GND
- D19 pad 2: Net-(D115-Pad2) -> +5V
- D19 pad 5: Net-(D115-Pad5) -> GND
- D190 pad 2: Net-(D110-Pad2) -> +5V
- D190 pad 5: Net-(D110-Pad5) -> GND
- D191 pad 2: Net-(D111-Pad2) -> +5V
- D191 pad 5: Net-(D111-Pad5) -> GND
- D192 pad 2: Net-(D112-Pad2) -> +5V
- D192 pad 5: Net-(D112-Pad5) -> GND
- D193 pad 2: Net-(D1-Pad2) -> +5V
- D193 pad 5: Net-(D1-Pad5) -> GND
- D194 pad 2: Net-(D114-Pad2) -> +5V
- D194 pad 5: Net-(D114-Pad5) -> GND
- D195 pad 2: Net-(D115-Pad2) -> +5V
- D195 pad 5: Net-(D115-Pad5) -> GND
- D196 pad 2: Net-(D100-Pad2) -> +5V
- D196 pad 5: Net-(D100-Pad5) -> GND
- D197 pad 2: Net-(D101-Pad2) -> +5V
- D197 pad 5: Net-(D101-Pad5) -> GND
- D198 pad 2: Net-(D102-Pad2) -> +5V
- D198 pad 5: Net-(D102-Pad5) -> GND
- D199 pad 2: Net-(D103-Pad2) -> +5V
- D199 pad 5: Net-(D103-Pad5) -> GND
- D2 pad 2: Net-(D114-Pad2) -> +5V
- D2 pad 5: Net-(D114-Pad5) -> GND
- D20 pad 2: Net-(D100-Pad2) -> +5V
- D20 pad 5: Net-(D100-Pad5) -> GND
- D200 pad 2: Net-(D104-Pad2) -> +5V
- D200 pad 5: Net-(D104-Pad5) -> GND
- D201 pad 2: Net-(D105-Pad2) -> +5V
- D201 pad 5: Net-(D105-Pad5) -> GND
- D202 pad 2: Net-(D10-Pad2) -> +5V
- D202 pad 5: Net-(D10-Pad5) -> GND
- D203 pad 2: Net-(D107-Pad2) -> +5V
- D203 pad 5: Net-(D107-Pad5) -> GND
- D204 pad 2: Net-(D108-Pad2) -> +5V
- D204 pad 5: Net-(D108-Pad5) -> GND
- D205 pad 2: Net-(D109-Pad2) -> +5V
- D205 pad 5: Net-(D109-Pad5) -> GND
- D206 pad 2: Net-(D110-Pad2) -> +5V
- D206 pad 5: Net-(D110-Pad5) -> GND
- D207 pad 2: Net-(D111-Pad2) -> +5V
- D207 pad 5: Net-(D111-Pad5) -> GND
- D208 pad 2: Net-(D112-Pad2) -> +5V
- D208 pad 5: Net-(D112-Pad5) -> GND
- D209 pad 2: Net-(D1-Pad2) -> +5V
- D209 pad 5: Net-(D1-Pad5) -> GND
- D21 pad 2: Net-(D101-Pad2) -> +5V
- D21 pad 5: Net-(D101-Pad5) -> GND
- D210 pad 2: Net-(D114-Pad2) -> +5V
- D210 pad 5: Net-(D114-Pad5) -> GND
- D211 pad 2: Net-(D115-Pad2) -> +5V
- D211 pad 5: Net-(D115-Pad5) -> GND
- D212 pad 2: Net-(D100-Pad2) -> +5V
- D212 pad 5: Net-(D100-Pad5) -> GND
- D213 pad 2: Net-(D101-Pad2) -> +5V
- D213 pad 5: Net-(D101-Pad5) -> GND
- D214 pad 2: Net-(D102-Pad2) -> +5V
- D214 pad 5: Net-(D102-Pad5) -> GND
- D215 pad 2: Net-(D103-Pad2) -> +5V
- D215 pad 5: Net-(D103-Pad5) -> GND
- D216 pad 2: Net-(D104-Pad2) -> +5V
- D216 pad 5: Net-(D104-Pad5) -> GND
- D217 pad 2: Net-(D105-Pad2) -> +5V
- D217 pad 5: Net-(D105-Pad5) -> GND
- D218 pad 2: Net-(D10-Pad2) -> +5V
- D218 pad 5: Net-(D10-Pad5) -> GND
- D219 pad 2: Net-(D107-Pad2) -> +5V
- D219 pad 5: Net-(D107-Pad5) -> GND
- D22 pad 2: Net-(D102-Pad2) -> +5V
- D22 pad 5: Net-(D102-Pad5) -> GND
- D220 pad 2: Net-(D108-Pad2) -> +5V
- D220 pad 5: Net-(D108-Pad5) -> GND
- D221 pad 2: Net-(D109-Pad2) -> +5V
- D221 pad 5: Net-(D109-Pad5) -> GND
- D222 pad 2: Net-(D110-Pad2) -> +5V
- D222 pad 5: Net-(D110-Pad5) -> GND
- D223 pad 2: Net-(D111-Pad2) -> +5V
- D223 pad 5: Net-(D111-Pad5) -> GND
- D224 pad 2: Net-(D112-Pad2) -> +5V
- D224 pad 5: Net-(D112-Pad5) -> GND
- D225 pad 2: Net-(D1-Pad2) -> +5V
- D225 pad 5: Net-(D1-Pad5) -> GND
- D226 pad 2: Net-(D114-Pad2) -> +5V
- D226 pad 5: Net-(D114-Pad5) -> GND
- D227 pad 2: Net-(D115-Pad2) -> +5V
- D227 pad 5: Net-(D115-Pad5) -> GND
- D228 pad 2: Net-(D100-Pad2) -> +5V
- D228 pad 5: Net-(D100-Pad5) -> GND
- D229 pad 2: Net-(D101-Pad2) -> +5V
- D229 pad 5: Net-(D101-Pad5) -> GND
- D23 pad 2: Net-(D103-Pad2) -> +5V
- D23 pad 5: Net-(D103-Pad5) -> GND
- D230 pad 2: Net-(D102-Pad2) -> +5V
- D230 pad 5: Net-(D102-Pad5) -> GND
- D231 pad 2: Net-(D103-Pad2) -> +5V
- D231 pad 5: Net-(D103-Pad5) -> GND
- D232 pad 2: Net-(D104-Pad2) -> +5V
- D232 pad 5: Net-(D104-Pad5) -> GND
- D233 pad 2: Net-(D105-Pad2) -> +5V
- D233 pad 5: Net-(D105-Pad5) -> GND
- D234 pad 2: Net-(D10-Pad2) -> +5V
- D234 pad 5: Net-(D10-Pad5) -> GND
- D235 pad 2: Net-(D107-Pad2) -> +5V
- D235 pad 5: Net-(D107-Pad5) -> GND
- D236 pad 2: Net-(D108-Pad2) -> +5V
- D236 pad 5: Net-(D108-Pad5) -> GND
- D237 pad 2: Net-(D109-Pad2) -> +5V
- D237 pad 5: Net-(D109-Pad5) -> GND
- D238 pad 2: Net-(D110-Pad2) -> +5V
- D238 pad 5: Net-(D110-Pad5) -> GND
- D239 pad 2: Net-(D111-Pad2) -> +5V
- D239 pad 5: Net-(D111-Pad5) -> GND
- D24 pad 2: Net-(D104-Pad2) -> +5V
- D24 pad 5: Net-(D104-Pad5) -> GND
- D240 pad 2: Net-(D112-Pad2) -> +5V
- D240 pad 5: Net-(D112-Pad5) -> GND
- D241 pad 2: Net-(D1-Pad2) -> +5V
- D241 pad 5: Net-(D1-Pad5) -> GND
- D242 pad 2: Net-(D114-Pad2) -> +5V
- D242 pad 5: Net-(D114-Pad5) -> GND
- D243 pad 2: Net-(D115-Pad2) -> +5V
- D243 pad 5: Net-(D115-Pad5) -> GND
- D244 pad 2: Net-(D100-Pad2) -> +5V
- D244 pad 5: Net-(D100-Pad5) -> GND
- D245 pad 2: Net-(D101-Pad2) -> +5V
- D245 pad 5: Net-(D101-Pad5) -> GND
- D246 pad 2: Net-(D102-Pad2) -> +5V
- D246 pad 5: Net-(D102-Pad5) -> GND
- D247 pad 2: Net-(D103-Pad2) -> +5V
- D247 pad 5: Net-(D103-Pad5) -> GND
- D248 pad 2: Net-(D104-Pad2) -> +5V
- D248 pad 5: Net-(D104-Pad5) -> GND
- D249 pad 2: Net-(D105-Pad2) -> +5V
- D249 pad 5: Net-(D105-Pad5) -> GND
- D25 pad 2: Net-(D105-Pad2) -> +5V
- D25 pad 5: Net-(D105-Pad5) -> GND
- D250 pad 2: Net-(D10-Pad2) -> +5V
- D250 pad 5: Net-(D10-Pad5) -> GND
- D251 pad 2: Net-(D107-Pad2) -> +5V
- D251 pad 5: Net-(D107-Pad5) -> GND
- D252 pad 2: Net-(D108-Pad2) -> +5V
- D252 pad 5: Net-(D108-Pad5) -> GND
- D253 pad 2: Net-(D109-Pad2) -> +5V
- D253 pad 5: Net-(D109-Pad5) -> GND
- D254 pad 2: Net-(D110-Pad2) -> +5V
- D254 pad 5: Net-(D110-Pad5) -> GND
- D255 pad 2: Net-(D111-Pad2) -> +5V
- D255 pad 5: Net-(D111-Pad5) -> GND
- D256 pad 2: Net-(D112-Pad2) -> +5V
- D256 pad 5: Net-(D112-Pad5) -> GND
- D26 pad 2: Net-(D10-Pad2) -> +5V
- D26 pad 5: Net-(D10-Pad5) -> GND
- D27 pad 2: Net-(D107-Pad2) -> +5V
- D27 pad 5: Net-(D107-Pad5) -> GND
- D28 pad 2: Net-(D108-Pad2) -> +5V
- D28 pad 5: Net-(D108-Pad5) -> GND
- D29 pad 2: Net-(D109-Pad2) -> +5V
- D29 pad 5: Net-(D109-Pad5) -> GND
- D3 pad 2: Net-(D115-Pad2) -> +5V
- D3 pad 5: Net-(D115-Pad5) -> GND
- D30 pad 2: Net-(D110-Pad2) -> +5V
- D30 pad 5: Net-(D110-Pad5) -> GND
- D31 pad 2: Net-(D111-Pad2) -> +5V
- D31 pad 5: Net-(D111-Pad5) -> GND
- D32 pad 2: Net-(D112-Pad2) -> +5V
- D32 pad 5: Net-(D112-Pad5) -> GND
- D33 pad 2: Net-(D1-Pad2) -> +5V
- D33 pad 5: Net-(D1-Pad5) -> GND
- D34 pad 2: Net-(D114-Pad2) -> +5V
- D34 pad 5: Net-(D114-Pad5) -> GND
- D35 pad 2: Net-(D115-Pad2) -> +5V
- D35 pad 5: Net-(D115-Pad5) -> GND
- D36 pad 2: Net-(D100-Pad2) -> +5V
- D36 pad 5: Net-(D100-Pad5) -> GND
- D37 pad 2: Net-(D101-Pad2) -> +5V
- D37 pad 5: Net-(D101-Pad5) -> GND
- D38 pad 2: Net-(D102-Pad2) -> +5V
- D38 pad 5: Net-(D102-Pad5) -> GND
- D39 pad 2: Net-(D103-Pad2) -> +5V
- D39 pad 5: Net-(D103-Pad5) -> GND
- D4 pad 2: Net-(D100-Pad2) -> +5V
- D4 pad 5: Net-(D100-Pad5) -> GND
- D40 pad 2: Net-(D104-Pad2) -> +5V
- D40 pad 5: Net-(D104-Pad5) -> GND
- D41 pad 2: Net-(D105-Pad2) -> +5V
- D41 pad 5: Net-(D105-Pad5) -> GND
- D42 pad 2: Net-(D10-Pad2) -> +5V
- D42 pad 5: Net-(D10-Pad5) -> GND
- D43 pad 2: Net-(D107-Pad2) -> +5V
- D43 pad 5: Net-(D107-Pad5) -> GND
- D44 pad 2: Net-(D108-Pad2) -> +5V
- D44 pad 5: Net-(D108-Pad5) -> GND
- D45 pad 2: Net-(D109-Pad2) -> +5V
- D45 pad 5: Net-(D109-Pad5) -> GND
- D46 pad 2: Net-(D110-Pad2) -> +5V
- D46 pad 5: Net-(D110-Pad5) -> GND
- D47 pad 2: Net-(D111-Pad2) -> +5V
- D47 pad 5: Net-(D111-Pad5) -> GND
- D48 pad 2: Net-(D112-Pad2) -> +5V
- D48 pad 5: Net-(D112-Pad5) -> GND
- D49 pad 2: Net-(D1-Pad2) -> +5V
- D49 pad 5: Net-(D1-Pad5) -> GND
- D5 pad 2: Net-(D101-Pad2) -> +5V
- D5 pad 5: Net-(D101-Pad5) -> GND
- D50 pad 2: Net-(D114-Pad2) -> +5V
- D50 pad 5: Net-(D114-Pad5) -> GND
- D51 pad 2: Net-(D115-Pad2) -> +5V
- D51 pad 5: Net-(D115-Pad5) -> GND
- D52 pad 2: Net-(D100-Pad2) -> +5V
- D52 pad 5: Net-(D100-Pad5) -> GND
- D53 pad 2: Net-(D101-Pad2) -> +5V
- D53 pad 5: Net-(D101-Pad5) -> GND
- D54 pad 2: Net-(D102-Pad2) -> +5V
- D54 pad 5: Net-(D102-Pad5) -> GND
- D55 pad 2: Net-(D103-Pad2) -> +5V
- D55 pad 5: Net-(D103-Pad5) -> GND
- D56 pad 2: Net-(D104-Pad2) -> +5V
- D56 pad 5: Net-(D104-Pad5) -> GND
- D57 pad 2: Net-(D105-Pad2) -> +5V
- D57 pad 5: Net-(D105-Pad5) -> GND
- D58 pad 2: Net-(D10-Pad2) -> +5V
- D58 pad 5: Net-(D10-Pad5) -> GND
- D59 pad 2: Net-(D107-Pad2) -> +5V
- D59 pad 5: Net-(D107-Pad5) -> GND
- D6 pad 2: Net-(D102-Pad2) -> +5V
- D6 pad 5: Net-(D102-Pad5) -> GND
- D60 pad 2: Net-(D108-Pad2) -> +5V
- D60 pad 5: Net-(D108-Pad5) -> GND
- D61 pad 2: Net-(D109-Pad2) -> +5V
- D61 pad 5: Net-(D109-Pad5) -> GND
- D62 pad 2: Net-(D110-Pad2) -> +5V
- D62 pad 5: Net-(D110-Pad5) -> GND
- D63 pad 2: Net-(D111-Pad2) -> +5V
- D63 pad 5: Net-(D111-Pad5) -> GND
- D64 pad 2: Net-(D112-Pad2) -> +5V
- D64 pad 5: Net-(D112-Pad5) -> GND
- D65 pad 2: Net-(D1-Pad2) -> +5V
- D65 pad 5: Net-(D1-Pad5) -> GND
- D66 pad 2: Net-(D114-Pad2) -> +5V
- D66 pad 5: Net-(D114-Pad5) -> GND
- D67 pad 2: Net-(D115-Pad2) -> +5V
- D67 pad 5: Net-(D115-Pad5) -> GND
- D68 pad 2: Net-(D100-Pad2) -> +5V
- D68 pad 5: Net-(D100-Pad5) -> GND
- D69 pad 2: Net-(D101-Pad2) -> +5V
- D69 pad 5: Net-(D101-Pad5) -> GND
- D7 pad 2: Net-(D103-Pad2) -> +5V
- D7 pad 5: Net-(D103-Pad5) -> GND
- D70 pad 2: Net-(D102-Pad2) -> +5V
- D70 pad 5: Net-(D102-Pad5) -> GND
- D71 pad 2: Net-(D103-Pad2) -> +5V
- D71 pad 5: Net-(D103-Pad5) -> GND
- D72 pad 2: Net-(D104-Pad2) -> +5V
- D72 pad 5: Net-(D104-Pad5) -> GND
- D73 pad 2: Net-(D105-Pad2) -> +5V
- D73 pad 5: Net-(D105-Pad5) -> GND
- D74 pad 2: Net-(D10-Pad2) -> +5V
- D74 pad 5: Net-(D10-Pad5) -> GND
- D75 pad 2: Net-(D107-Pad2) -> +5V
- D75 pad 5: Net-(D107-Pad5) -> GND
- D76 pad 2: Net-(D108-Pad2) -> +5V
- D76 pad 5: Net-(D108-Pad5) -> GND
- D77 pad 2: Net-(D109-Pad2) -> +5V
- D77 pad 5: Net-(D109-Pad5) -> GND
- D78 pad 2: Net-(D110-Pad2) -> +5V
- D78 pad 5: Net-(D110-Pad5) -> GND
- D79 pad 2: Net-(D111-Pad2) -> +5V
- D79 pad 5: Net-(D111-Pad5) -> GND
- D8 pad 2: Net-(D104-Pad2) -> +5V
- D8 pad 5: Net-(D104-Pad5) -> GND
- D80 pad 2: Net-(D112-Pad2) -> +5V
- D80 pad 5: Net-(D112-Pad5) -> GND
- D81 pad 2: Net-(D1-Pad2) -> +5V
- D81 pad 5: Net-(D1-Pad5) -> GND
- D82 pad 2: Net-(D114-Pad2) -> +5V
- D82 pad 5: Net-(D114-Pad5) -> GND
- D83 pad 2: Net-(D115-Pad2) -> +5V
- D83 pad 5: Net-(D115-Pad5) -> GND
- D84 pad 2: Net-(D100-Pad2) -> +5V
- D84 pad 5: Net-(D100-Pad5) -> GND
- D85 pad 2: Net-(D101-Pad2) -> +5V
- D85 pad 5: Net-(D101-Pad5) -> GND
- D86 pad 2: Net-(D102-Pad2) -> +5V
- D86 pad 5: Net-(D102-Pad5) -> GND
- D87 pad 2: Net-(D103-Pad2) -> +5V
- D87 pad 5: Net-(D103-Pad5) -> GND
- D88 pad 2: Net-(D104-Pad2) -> +5V
- D88 pad 5: Net-(D104-Pad5) -> GND
- D89 pad 2: Net-(D105-Pad2) -> +5V
- D89 pad 5: Net-(D105-Pad5) -> GND
- D9 pad 2: Net-(D105-Pad2) -> +5V
- D9 pad 5: Net-(D105-Pad5) -> GND
- D90 pad 2: Net-(D10-Pad2) -> +5V
- D90 pad 5: Net-(D10-Pad5) -> GND
- D91 pad 2: Net-(D107-Pad2) -> +5V
- D91 pad 5: Net-(D107-Pad5) -> GND
- D92 pad 2: Net-(D108-Pad2) -> +5V
- D92 pad 5: Net-(D108-Pad5) -> GND
- D93 pad 2: Net-(D109-Pad2) -> +5V
- D93 pad 5: Net-(D109-Pad5) -> GND
- D94 pad 2: Net-(D110-Pad2) -> +5V
- D94 pad 5: Net-(D110-Pad5) -> GND
- D95 pad 2: Net-(D111-Pad2) -> +5V
- D95 pad 5: Net-(D111-Pad5) -> GND
- D96 pad 2: Net-(D112-Pad2) -> +5V
- D96 pad 5: Net-(D112-Pad5) -> GND
- D97 pad 2: Net-(D1-Pad2) -> +5V
- D97 pad 5: Net-(D1-Pad5) -> GND
- D98 pad 2: Net-(D114-Pad2) -> +5V
- D98 pad 5: Net-(D114-Pad5) -> GND
- D99 pad 2: Net-(D115-Pad2) -> +5V
- D99 pad 5: Net-(D115-Pad5) -> GND
- H1 pad 1: Net-(H1-Pad1) -> GND
- H2 pad 1: Net-(H2-Pad1) -> GND
- H3 pad 1: Net-(H3-Pad1) -> GND
- H4 pad 1: Net-(H4-Pad1) -> GND
- R1 pad 1: Net-(D1-Pad2) -> +5V
- R10 pad 1: Net-(D10-Pad2) -> +5V
- R100 pad 1: Net-(D100-Pad2) -> +5V
- R101 pad 1: Net-(D101-Pad2) -> +5V
- R102 pad 1: Net-(D102-Pad2) -> +5V
- R103 pad 1: Net-(D103-Pad2) -> +5V
- R104 pad 1: Net-(D104-Pad2) -> +5V
- R105 pad 1: Net-(D105-Pad2) -> +5V
- R106 pad 1: Net-(D10-Pad2) -> +5V
- R107 pad 1: Net-(D107-Pad2) -> +5V
- R108 pad 1: Net-(D108-Pad2) -> +5V
- R109 pad 1: Net-(D109-Pad2) -> +5V
- R11 pad 1: Net-(D107-Pad2) -> +5V
- R110 pad 1: Net-(D110-Pad2) -> +5V
- R111 pad 1: Net-(D111-Pad2) -> +5V
- R112 pad 1: Net-(D112-Pad2) -> +5V
- R113 pad 1: Net-(D1-Pad2) -> +5V
- R114 pad 1: Net-(D114-Pad2) -> +5V
- R115 pad 1: Net-(D115-Pad2) -> +5V
- R116 pad 1: Net-(D100-Pad2) -> +5V
- R117 pad 1: Net-(D101-Pad2) -> +5V
- R118 pad 1: Net-(D102-Pad2) -> +5V
- R119 pad 1: Net-(D103-Pad2) -> +5V
- R12 pad 1: Net-(D108-Pad2) -> +5V
- R120 pad 1: Net-(D104-Pad2) -> +5V
- R121 pad 1: Net-(D105-Pad2) -> +5V
- R122 pad 1: Net-(D10-Pad2) -> +5V
- R123 pad 1: Net-(D107-Pad2) -> +5V
- R124 pad 1: Net-(D108-Pad2) -> +5V
- R125 pad 1: Net-(D109-Pad2) -> +5V
- R126 pad 1: Net-(D110-Pad2) -> +5V
- R127 pad 1: Net-(D111-Pad2) -> +5V
- R128 pad 1: Net-(D112-Pad2) -> +5V
- R129 pad 1: Net-(D1-Pad2) -> +5V
- R13 pad 1: Net-(D109-Pad2) -> +5V
- R130 pad 1: Net-(D114-Pad2) -> +5V
- R131 pad 1: Net-(D115-Pad2) -> +5V
- R132 pad 1: Net-(D100-Pad2) -> +5V
- R133 pad 1: Net-(D101-Pad2) -> +5V
- R134 pad 1: Net-(D102-Pad2) -> +5V
- R135 pad 1: Net-(D103-Pad2) -> +5V
- R136 pad 1: Net-(D104-Pad2) -> +5V
- R137 pad 1: Net-(D105-Pad2) -> +5V
- R138 pad 1: Net-(D10-Pad2) -> +5V
- R139 pad 1: Net-(D107-Pad2) -> +5V
- R14 pad 1: Net-(D110-Pad2) -> +5V
- R140 pad 1: Net-(D108-Pad2) -> +5V
- R141 pad 1: Net-(D109-Pad2) -> +5V
- R142 pad 1: Net-(D110-Pad2) -> +5V
- R143 pad 1: Net-(D111-Pad2) -> +5V
- R144 pad 1: Net-(D112-Pad2) -> +5V
- R145 pad 1: Net-(D1-Pad2) -> +5V
- R146 pad 1: Net-(D114-Pad2) -> +5V
- R147 pad 1: Net-(D115-Pad2) -> +5V
- R148 pad 1: Net-(D100-Pad2) -> +5V
- R149 pad 1: Net-(D101-Pad2) -> +5V
- R15 pad 1: Net-(D111-Pad2) -> +5V
- R150 pad 1: Net-(D102-Pad2) -> +5V
- R151 pad 1: Net-(D103-Pad2) -> +5V
- R152 pad 1: Net-(D104-Pad2) -> +5V
- R153 pad 1: Net-(D105-Pad2) -> +5V
- R154 pad 1: Net-(D10-Pad2) -> +5V
- R155 pad 1: Net-(D107-Pad2) -> +5V
- R156 pad 1: Net-(D108-Pad2) -> +5V
- R157 pad 1: Net-(D109-Pad2) -> +5V
- R158 pad 1: Net-(D110-Pad2) -> +5V
- R159 pad 1: Net-(D111-Pad2) -> +5V
- R16 pad 1: Net-(D112-Pad2) -> +5V
- R160 pad 1: Net-(D112-Pad2) -> +5V
- R161 pad 1: Net-(D1-Pad2) -> +5V
- R162 pad 1: Net-(D114-Pad2) -> +5V
- R163 pad 1: Net-(D115-Pad2) -> +5V
- R164 pad 1: Net-(D100-Pad2) -> +5V
- R165 pad 1: Net-(D101-Pad2) -> +5V
- R166 pad 1: Net-(D102-Pad2) -> +5V
- R167 pad 1: Net-(D103-Pad2) -> +5V
- R168 pad 1: Net-(D104-Pad2) -> +5V
- R169 pad 1: Net-(D105-Pad2) -> +5V
- R17 pad 1: Net-(D1-Pad2) -> +5V
- R170 pad 1: Net-(D10-Pad2) -> +5V
- R171 pad 1: Net-(D107-Pad2) -> +5V
- R172 pad 1: Net-(D108-Pad2) -> +5V
- R173 pad 1: Net-(D109-Pad2) -> +5V
- R174 pad 1: Net-(D110-Pad2) -> +5V
- R175 pad 1: Net-(D111-Pad2) -> +5V
- R176 pad 1: Net-(D112-Pad2) -> +5V
- R177 pad 1: Net-(D1-Pad2) -> +5V
- R178 pad 1: Net-(D114-Pad2) -> +5V
- R179 pad 1: Net-(D115-Pad2) -> +5V
- R18 pad 1: Net-(D114-Pad2) -> +5V
- R180 pad 1: Net-(D100-Pad2) -> +5V
- R181 pad 1: Net-(D101-Pad2) -> +5V
- R182 pad 1: Net-(D102-Pad2) -> +5V
- R183 pad 1: Net-(D103-Pad2) -> +5V
- R184 pad 1: Net-(D104-Pad2) -> +5V
- R185 pad 1: Net-(D105-Pad2) -> +5V
- R186 pad 1: Net-(D10-Pad2) -> +5V
- R187 pad 1: Net-(D107-Pad2) -> +5V
- R188 pad 1: Net-(D108-Pad2) -> +5V
- R189 pad 1: Net-(D109-Pad2) -> +5V
- R19 pad 1: Net-(D115-Pad2) -> +5V
- R190 pad 1: Net-(D110-Pad2) -> +5V
- R191 pad 1: Net-(D111-Pad2) -> +5V
- R192 pad 1: Net-(D112-Pad2) -> +5V
- R193 pad 1: Net-(D1-Pad2) -> +5V
- R194 pad 1: Net-(D114-Pad2) -> +5V
- R195 pad 1: Net-(D115-Pad2) -> +5V
- R196 pad 1: Net-(D100-Pad2) -> +5V
- R197 pad 1: Net-(D101-Pad2) -> +5V
- R198 pad 1: Net-(D102-Pad2) -> +5V
- R199 pad 1: Net-(D103-Pad2) -> +5V
- R2 pad 1: Net-(D114-Pad2) -> +5V
- R20 pad 1: Net-(D100-Pad2) -> +5V
- R200 pad 1: Net-(D104-Pad2) -> +5V
- R201 pad 1: Net-(D105-Pad2) -> +5V
- R202 pad 1: Net-(D10-Pad2) -> +5V
- R203 pad 1: Net-(D107-Pad2) -> +5V
- R204 pad 1: Net-(D108-Pad2) -> +5V
- R205 pad 1: Net-(D109-Pad2) -> +5V
- R206 pad 1: Net-(D110-Pad2) -> +5V
- R207 pad 1: Net-(D111-Pad2) -> +5V
- R208 pad 1: Net-(D112-Pad2) -> +5V
- R209 pad 1: Net-(D1-Pad2) -> +5V
- R21 pad 1: Net-(D101-Pad2) -> +5V
- R210 pad 1: Net-(D114-Pad2) -> +5V
- R211 pad 1: Net-(D115-Pad2) -> +5V
- R212 pad 1: Net-(D100-Pad2) -> +5V
- R213 pad 1: Net-(D101-Pad2) -> +5V
- R214 pad 1: Net-(D102-Pad2) -> +5V
- R215 pad 1: Net-(D103-Pad2) -> +5V
- R216 pad 1: Net-(D104-Pad2) -> +5V
- R217 pad 1: Net-(D105-Pad2) -> +5V
- R218 pad 1: Net-(D10-Pad2) -> +5V
- R219 pad 1: Net-(D107-Pad2) -> +5V
- R22 pad 1: Net-(D102-Pad2) -> +5V
- R220 pad 1: Net-(D108-Pad2) -> +5V
- R221 pad 1: Net-(D109-Pad2) -> +5V
- R222 pad 1: Net-(D110-Pad2) -> +5V
- R223 pad 1: Net-(D111-Pad2) -> +5V
- R224 pad 1: Net-(D112-Pad2) -> +5V
- R225 pad 1: Net-(D1-Pad2) -> +5V
- R226 pad 1: Net-(D114-Pad2) -> +5V
- R227 pad 1: Net-(D115-Pad2) -> +5V
- R228 pad 1: Net-(D100-Pad2) -> +5V
- R229 pad 1: Net-(D101-Pad2) -> +5V
- R23 pad 1: Net-(D103-Pad2) -> +5V
- R230 pad 1: Net-(D102-Pad2) -> +5V
- R231 pad 1: Net-(D103-Pad2) -> +5V
- R232 pad 1: Net-(D104-Pad2) -> +5V
- R233 pad 1: Net-(D105-Pad2) -> +5V
- R234 pad 1: Net-(D10-Pad2) -> +5V
- R235 pad 1: Net-(D107-Pad2) -> +5V
- R236 pad 1: Net-(D108-Pad2) -> +5V
- R237 pad 1: Net-(D109-Pad2) -> +5V
- R238 pad 1: Net-(D110-Pad2) -> +5V
- R239 pad 1: Net-(D111-Pad2) -> +5V
- R24 pad 1: Net-(D104-Pad2) -> +5V
- R240 pad 1: Net-(D112-Pad2) -> +5V
- R241 pad 1: Net-(D1-Pad2) -> +5V
- R242 pad 1: Net-(D114-Pad2) -> +5V
- R243 pad 1: Net-(D115-Pad2) -> +5V
- R244 pad 1: Net-(D100-Pad2) -> +5V
- R245 pad 1: Net-(D101-Pad2) -> +5V
- R246 pad 1: Net-(D102-Pad2) -> +5V
- R247 pad 1: Net-(D103-Pad2) -> +5V
- R248 pad 1: Net-(D104-Pad2) -> +5V
- R249 pad 1: Net-(D105-Pad2) -> +5V
- R25 pad 1: Net-(D105-Pad2) -> +5V
- R250 pad 1: Net-(D10-Pad2) -> +5V
- R251 pad 1: Net-(D107-Pad2) -> +5V
- R252 pad 1: Net-(D108-Pad2) -> +5V
- R253 pad 1: Net-(D109-Pad2) -> +5V
- R254 pad 1: Net-(D110-Pad2) -> +5V
- R255 pad 1: Net-(D111-Pad2) -> +5V
- R256 pad 1: Net-(D112-Pad2) -> +5V
- R26 pad 1: Net-(D10-Pad2) -> +5V
- R27 pad 1: Net-(D107-Pad2) -> +5V
- R28 pad 1: Net-(D108-Pad2) -> +5V
- R29 pad 1: Net-(D109-Pad2) -> +5V
- R3 pad 1: Net-(D115-Pad2) -> +5V
- R30 pad 1: Net-(D110-Pad2) -> +5V
- R31 pad 1: Net-(D111-Pad2) -> +5V
- R32 pad 1: Net-(D112-Pad2) -> +5V
- R33 pad 1: Net-(D1-Pad2) -> +5V
- R34 pad 1: Net-(D114-Pad2) -> +5V
- R35 pad 1: Net-(D115-Pad2) -> +5V
- R36 pad 1: Net-(D100-Pad2) -> +5V
- R37 pad 1: Net-(D101-Pad2) -> +5V
- R38 pad 1: Net-(D102-Pad2) -> +5V
- R39 pad 1: Net-(D103-Pad2) -> +5V
- R4 pad 1: Net-(D100-Pad2) -> +5V
- R40 pad 1: Net-(D104-Pad2) -> +5V
- R41 pad 1: Net-(D105-Pad2) -> +5V
- R42 pad 1: Net-(D10-Pad2) -> +5V
- R43 pad 1: Net-(D107-Pad2) -> +5V
- R44 pad 1: Net-(D108-Pad2) -> +5V
- R45 pad 1: Net-(D109-Pad2) -> +5V
- R46 pad 1: Net-(D110-Pad2) -> +5V
- R47 pad 1: Net-(D111-Pad2) -> +5V
- R48 pad 1: Net-(D112-Pad2) -> +5V
- R49 pad 1: Net-(D1-Pad2) -> +5V
- R5 pad 1: Net-(D101-Pad2) -> +5V
- R50 pad 1: Net-(D114-Pad2) -> +5V
- R51 pad 1: Net-(D115-Pad2) -> +5V
- R52 pad 1: Net-(D100-Pad2) -> +5V
- R53 pad 1: Net-(D101-Pad2) -> +5V
- R54 pad 1: Net-(D102-Pad2) -> +5V
- R55 pad 1: Net-(D103-Pad2) -> +5V
- R56 pad 1: Net-(D104-Pad2) -> +5V
- R57 pad 1: Net-(D105-Pad2) -> +5V
- R58 pad 1: Net-(D10-Pad2) -> +5V
- R59 pad 1: Net-(D107-Pad2) -> +5V
- R6 pad 1: Net-(D102-Pad2) -> +5V
- R60 pad 1: Net-(D108-Pad2) -> +5V
- R61 pad 1: Net-(D109-Pad2) -> +5V
- R62 pad 1: Net-(D110-Pad2) -> +5V
- R63 pad 1: Net-(D111-Pad2) -> +5V
- R64 pad 1: Net-(D112-Pad2) -> +5V
- R65 pad 1: Net-(D1-Pad2) -> +5V
- R66 pad 1: Net-(D114-Pad2) -> +5V
- R67 pad 1: Net-(D115-Pad2) -> +5V
- R68 pad 1: Net-(D100-Pad2) -> +5V
- R69 pad 1: Net-(D101-Pad2) -> +5V
- R7 pad 1: Net-(D103-Pad2) -> +5V
- R70 pad 1: Net-(D102-Pad2) -> +5V
- R71 pad 1: Net-(D103-Pad2) -> +5V
- R72 pad 1: Net-(D104-Pad2) -> +5V
- R73 pad 1: Net-(D105-Pad2) -> +5V
- R74 pad 1: Net-(D10-Pad2) -> +5V
- R75 pad 1: Net-(D107-Pad2) -> +5V
- R76 pad 1: Net-(D108-Pad2) -> +5V
- R77 pad 1: Net-(D109-Pad2) -> +5V
- R78 pad 1: Net-(D110-Pad2) -> +5V
- R79 pad 1: Net-(D111-Pad2) -> +5V
- R8 pad 1: Net-(D104-Pad2) -> +5V
- R80 pad 1: Net-(D112-Pad2) -> +5V
- R81 pad 1: Net-(D1-Pad2) -> +5V
- R82 pad 1: Net-(D114-Pad2) -> +5V
- R83 pad 1: Net-(D115-Pad2) -> +5V
- R84 pad 1: Net-(D100-Pad2) -> +5V
- R85 pad 1: Net-(D101-Pad2) -> +5V
- R86 pad 1: Net-(D102-Pad2) -> +5V
- R87 pad 1: Net-(D103-Pad2) -> +5V
- R88 pad 1: Net-(D104-Pad2) -> +5V
- R89 pad 1: Net-(D105-Pad2) -> +5V
- R9 pad 1: Net-(D105-Pad2) -> +5V
- R90 pad 1: Net-(D10-Pad2) -> +5V
- R91 pad 1: Net-(D107-Pad2) -> +5V
- R92 pad 1: Net-(D108-Pad2) -> +5V
- R93 pad 1: Net-(D109-Pad2) -> +5V
- R94 pad 1: Net-(D110-Pad2) -> +5V
- R95 pad 1: Net-(D111-Pad2) -> +5V
- R96 pad 1: Net-(D112-Pad2) -> +5V
- R97 pad 1: Net-(D1-Pad2) -> +5V
- R98 pad 1: Net-(D114-Pad2) -> +5V
- R99 pad 1: Net-(D115-Pad2) -> +5V
Routing:
- net +5V: track 0.00 -> 7684.8 mm, vias 0 -> 39
- net GND: track 0.00 -> 3819.2 mm, vias 0 -> 233
- net Net-(D226-Pad3): track 0.00 -> 265.9 mm, vias 0 -> 2
- net Net-(D20-Pad6): track 0.00 -> 251.8 mm, vias 0 -> 2
- net Net-(D19-Pad6): track 0.00 -> 246.7 mm, vias 0 -> 4
- net Net-(D18-Pad6): track 0.00 -> 239.1 mm, vias 0 -> 2
- net Net-(D2-Pad6): track 0.00 -> 238.1 mm, vias 0 -> 4
- net Net-(D15-Pad4): track 0.00 -> 237.8 mm, vias 0 -> 2
- net Net-(D23-Pad6): track 0.00 -> 236.6 mm, vias 0 -> 2
- net Net-(D21-Pad6): track 0.00 -> 234.7 mm, vias 0 -> 2
- net Net-(D229-Pad3): track 0.00 -> 234.2 mm, vias 0 -> 2
- net Net-(D227-Pad3): track 0.00 -> 234.0 mm, vias 0 -> 2
- net Net-(D22-Pad6): track 0.00 -> 233.8 mm, vias 0 -> 2
- net Net-(D228-Pad3): track 0.00 -> 233.0 mm, vias 0 -> 2
- net Net-(D14-Pad6): track 0.00 -> 226.0 mm, vias 0 -> 2
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- added copper zone on B.Cu, net GND
- added copper zone on F.Cu, net GND
Other:
- rule via_min_drill: 0.3 -> 0.2
- rule via_min_size: 0.4 -> 0.45
- board text added: "3V3"
- board text added: "5V"
- board text added: "DESIGNED BY K.K."
- board text added: "GPIO"
- board text added: "IN CANADA"
- board text added: "KALA MAIN LED PCB v2"
