File: hw/Main_LED_PCB_v2/main_led_pcb/main_led_pcb.sch (KiCad schematic (older format))
At the start: 539 parts, among them J1 PWR_IN, J2 AVR-ISP-6, J3 UART, J4 I2C, J5 PA, J6 PB, U1 ATtiny87-MU, U2 NCP1117-3.3_SOT223

Commit message: Add all files, sort out later
Parts:
- added C? (x256): 100n, Capacitor_SMD:C_0805_2012Metric_Pad1.15x1.40mm_HandSolder, symbol Device:C
- added J? (x3): PWR_IN, Connector_PinHeader_2.54mm:PinHeader_1x02_P2.54mm_Vertical, symbol Connector_Generic:Conn_01x02
- J3, J4: footprint Connector_PinHeader_2.54mm:PinHeader_1x02_P2.54mm_Vertical -> Connector_PinHeader_2.54mm:PinHeader_1x03_P2.54mm_Vertical; symbol Connector_Generic:Conn_01x02 -> Connector_Generic:Conn_01x03
Connections:
- net +5V: now also D1.2 (VDD), D10.2 (VDD), D100.2 (VDD), D101.2 (VDD), D102.2 (VDD), D103.2 (VDD), D104.2 (VDD), D105.2 (VDD), D106.2 (VDD), D107.2 (VDD), D108.2 (VDD), D109.2 (VDD), D11.2 (VDD), D110.2 (VDD), D111.2 (VDD), D112.2 (VDD), D113.2 (VDD), D114.2 (VDD), D115.2 (VDD), D116.2 (VDD), D117.2 (VDD), D118.2 (VDD), D119.2 (VDD), D12.2 (VDD), D120.2 (VDD), D121.2 (VDD), D122.2 (VDD), D123.2 (VDD), D124.2 (VDD), D125.2 (VDD), D126.2 (VDD), D127.2 (VDD), D128.2 (VDD), D129.2 (VDD), D13.2 (VDD), D130.2 (VDD), D131.2 (VDD), D132.2 (VDD), D133.2 (VDD), D134.2 (VDD), D135.2 (VDD), D136.2 (VDD), D137.2 (VDD), D138.2 (VDD), D139.2 (VDD), D14.2 (VDD), D140.2 (VDD), D141.2 (VDD), D142.2 (VDD), D143.2 (VDD), D144.2 (VDD), D145.2 (VDD), D146.2 (VDD), D147.2 (VDD), D148.2 (VDD), D149.2 (VDD), D15.2 (VDD), D150.2 (VDD), D151.2 (VDD), D152.2 (VDD), D153.2 (VDD), D154.2 (VDD), D155.2 (VDD), D156.2 (VDD), D157.2 (VDD), D158.2 (VDD), D159.2 (VDD), D16.2 (VDD), D160.2 (VDD), D161.2 (VDD), D162.2 (VDD), D163.2 (VDD), D164.2 (VDD), D165.2 (VDD), D166.2 (VDD), D167.2 (VDD), D168.2 (VDD), D169.2 (VDD), D17.2 (VDD), D170.2 (VDD), D171.2 (VDD), D172.2 (VDD), D173.2 (VDD), D174.2 (VDD), D175.2 (VDD), D176.2 (VDD), D177.2 (VDD), D178.2 (VDD), D179.2 (VDD), D18.2 (VDD), D180.2 (VDD), D181.2 (VDD), D182.2 (VDD), D183.2 (VDD), D184.2 (VDD), D185.2 (VDD), D186.2 (VDD), D187.2 (VDD), D188.2 (VDD), D189.2 (VDD), D19.2 (VDD), D190.2 (VDD), D191.2 (VDD), D192.2 (VDD), D193.2 (VDD), D194.2 (VDD), D195.2 (VDD), D196.2 (VDD), D197.2 (VDD), D198.2 (VDD), D199.2 (VDD), D2.2 (VDD), D20.2 (VDD), D200.2 (VDD), D201.2 (VDD), D202.2 (VDD), D203.2 (VDD), D204.2 (VDD), D205.2 (VDD), D206.2 (VDD), D207.2 (VDD), D208.2 (VDD), D209.2 (VDD), D21.2 (VDD), D210.2 (VDD), D211.2 (VDD), D212.2 (VDD), D213.2 (VDD), D214.2 (VDD), D215.2 (VDD), D216.2 (VDD), D217.2 (VDD), D218.2 (VDD), D219.2 (VDD), D22.2 (VDD), D220.2 (VDD), D221.2 (VDD), D222.2 (VDD), D223.2 (VDD), D224.2 (VDD), D225.2 (VDD), D226.2 (VDD), D227.2 (VDD), D228.2 (VDD), D229.2 (VDD), D23.2 (VDD), D230.2 (VDD), D231.2 (VDD), D232.2 (VDD), D233.2 (VDD), D234.2 (VDD), D235.2 (VDD), D236.2 (VDD), D237.2 (VDD), D238.2 (VDD), D239.2 (VDD), D24.2 (VDD), D240.2 (VDD), D241.2 (VDD), D242.2 (VDD), D243.2 (VDD), D244.2 (VDD), D245.2 (VDD), D246.2 (VDD), D247.2 (VDD), D248.2 (VDD), D249.2 (VDD), D25.2 (VDD), D250.2 (VDD), D251.2 (VDD), D252.2 (VDD), D253.2 (VDD), D254.2 (VDD), D255.2 (VDD), D256.2 (VDD), D26.2 (VDD), D27.2 (VDD), D28.2 (VDD), D29.2 (VDD), D3.2 (VDD), D30.2 (VDD), D31.2 (VDD), D32.2 (VDD), D33.2 (VDD), D34.2 (VDD), D35.2 (VDD), D36.2 (VDD), D37.2 (VDD), D38.2 (VDD), D39.2 (VDD), D4.2 (VDD), D40.2 (VDD), D41.2 (VDD), D42.2 (VDD), D43.2 (VDD), D44.2 (VDD), D45.2 (VDD), D46.2 (VDD), D47.2 (VDD), D48.2 (VDD), D49.2 (VDD), D5.2 (VDD), D50.2 (VDD), D51.2 (VDD), D52.2 (VDD), D53.2 (VDD), D54.2 (VDD), D55.2 (VDD), D56.2 (VDD), D57.2 (VDD), D58.2 (VDD), D59.2 (VDD), D6.2 (VDD), D60.2 (VDD), D61.2 (VDD), D62.2 (VDD), D63.2 (VDD), D64.2 (VDD), D65.2 (VDD), D66.2 (VDD), D67.2 (VDD), D68.2 (VDD), D69.2 (VDD), D7.2 (VDD), D70.2 (VDD), D71.2 (VDD), D72.2 (VDD), D73.2 (VDD), D74.2 (VDD), D75.2 (VDD), D76.2 (VDD), D77.2 (VDD), D78.2 (VDD), D79.2 (VDD), D8.2 (VDD), D80.2 (VDD), D81.2 (VDD), D82.2 (VDD), D83.2 (VDD), D84.2 (VDD), D85.2 (VDD), D86.2 (VDD), D87.2 (VDD), D88.2 (VDD), D89.2 (VDD), D9.2 (VDD), D90.2 (VDD), D91.2 (VDD), D92.2 (VDD), D93.2 (VDD), D94.2 (VDD), D95.2 (VDD), D96.2 (VDD), D97.2 (VDD), D98.2 (VDD), D99.2 (VDD), R1.1, R10.1, R100.1, R101.1, R102.1, R103.1, R104.1, R105.1, R106.1, R107.1, R108.1, R109.1, R11.1, R110.1, R111.1, R112.1, R113.1, R114.1, R115.1, R116.1, R117.1, R118.1, R119.1, R12.1, R120.1, R121.1, R122.1, R123.1, R124.1, R125.1, R126.1, R127.1, R128.1, R129.1, R13.1, R130.1, R131.1, R132.1, R133.1, R134.1, R135.1, R136.1, R137.1, R138.1, R139.1, R14.1, R140.1, R141.1, R142.1, R143.1, R144.1, R145.1, R146.1, R147.1, R148.1, R149.1, R15.1, R150.1, R151.1, R152.1, R153.1, R154.1, R155.1, R156.1, R157.1, R158.1, R159.1, R16.1, R160.1, R161.1, R162.1, R163.1, R164.1, R165.1, R166.1, R167.1, R168.1, R169.1, R17.1, R170.1, R171.1, R172.1, R173.1, R174.1, R175.1, R176.1, R177.1, R178.1, R179.1, R18.1, R180.1, R181.1, R182.1, R183.1, R184.1, R185.1, R186.1, R187.1, R188.1, R189.1, R19.1, R190.1, R191.1, R192.1, R193.1, R194.1, R195.1, R196.1, R197.1, R198.1, R199.1, R2.1, R20.1, R200.1, R201.1, R202.1, R203.1, R204.1, R205.1, R206.1, R207.1, R208.1, R209.1, R21.1, R210.1, R211.1, R212.1, R213.1, R214.1, R215.1, R216.1, R217.1, R218.1, R219.1, R22.1, R220.1, R221.1, R222.1, R223.1, R224.1, R225.1, R226.1, R227.1, R228.1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
- net GND: now also D1.5 (GND), D10.5 (GND), D100.5 (GND), D101.5 (GND), D102.5 (GND), D103.5 (GND), D104.5 (GND), D105.5 (GND), D106.5 (GND), D107.5 (GND), D108.5 (GND), D109.5 (GND), D11.5 (GND), D110.5 (GND), D111.5 (GND), D112.5 (GND), D113.5 (GND), D114.5 (GND), D115.5 (GND), D116.5 (GND), D117.5 (GND), D118.5 (GND), D119.5 (GND), D12.5 (GND), D120.5 (GND), D121.5 (GND), D122.5 (GND), D123.5 (GND), D124.5 (GND), D125.5 (GND), D126.5 (GND), D127.5 (GND), D128.5 (GND), D129.5 (GND), D13.5 (GND), D130.5 (GND), D131.5 (GND), D132.5 (GND), D133.5 (GND), D134.5 (GND), D135.5 (GND), D136.5 (GND), D137.5 (GND), D138.5 (GND), D139.5 (GND), D14.5 (GND), D140.5 (GND), D141.5 (GND), D142.5 (GND), D143.5 (GND), D144.5 (GND), D145.5 (GND), D146.5 (GND), D147.5 (GND), D148.5 (GND), D149.5 (GND), D15.5 (GND), D150.5 (GND), D151.5 (GND), D152.5 (GND), D153.5 (GND), D154.5 (GND), D155.5 (GND), D156.5 (GND), D157.5 (GND), D158.5 (GND), D159.5 (GND), D16.5 (GND), D160.5 (GND), D161.5 (GND), D162.5 (GND), D163.5 (GND), D164.5 (GND), D165.5 (GND), D166.5 (GND), D167.5 (GND), D168.5 (GND), D169.5 (GND), D17.5 (GND), D170.5 (GND), D171.5 (GND), D172.5 (GND), D173.5 (GND), D174.5 (GND), D175.5 (GND), D176.5 (GND), D177.5 (GND), D178.5 (GND), D179.5 (GND), D18.5 (GND), D180.5 (GND), D181.5 (GND), D182.5 (GND), D183.5 (GND), D184.5 (GND), D185.5 (GND), D186.5 (GND), D187.5 (GND), D188.5 (GND), D189.5 (GND), D19.5 (GND), D190.5 (GND), D191.5 (GND), D192.5 (GND), D193.5 (GND), D194.5 (GND), D195.5 (GND), D196.5 (GND), D197.5 (GND), D198.5 (GND), D199.5 (GND), D2.5 (GND), D20.5 (GND), D200.5 (GND), D201.5 (GND), D202.5 (GND), D203.5 (GND), D204.5 (GND), D205.5 (GND), D206.5 (GND), D207.5 (GND), D208.5 (GND), D209.5 (GND), D21.5 (GND), D210.5 (GND), D211.5 (GND), D212.5 (GND), D213.5 (GND), D214.5 (GND), D215.5 (GND), D216.5 (GND), D217.5 (GND), D218.5 (GND), D219.5 (GND), D22.5 (GND), D220.5 (GND), D221.5 (GND), D222.5 (GND), D223.5 (GND), D224.5 (GND), D225.5 (GND), D226.5 (GND), D227.5 (GND), D228.5 (GND), D229.5 (GND), D23.5 (GND), D230.5 (GND), D231.5 (GND), D232.5 (GND), D233.5 (GND), D234.5 (GND), D235.5 (GND), D236.5 (GND), D237.5 (GND), D238.5 (GND), D239.5 (GND), D24.5 (GND), D240.5 (GND), D241.5 (GND), D242.5 (GND), D243.5 (GND), D244.5 (GND), D245.5 (GND), D246.5 (GND), D247.5 (GND), D248.5 (GND), D249.5 (GND), D25.5 (GND), D250.5 (GND), D251.5 (GND), D252.5 (GND), D253.5 (GND), D254.5 (GND), D255.5 (GND), D256.5 (GND), D26.5 (GND), D27.5 (GND), D28.5 (GND), D29.5 (GND), D3.5 (GND), D30.5 (GND), D31.5 (GND), D32.5 (GND), D33.5 (GND), D34.5 (GND), D35.5 (GND), D36.5 (GND), D37.5 (GND), D38.5 (GND), D39.5 (GND), D4.5 (GND), D40.5 (GND), D41.5 (GND), D42.5 (GND), D43.5 (GND), D44.5 (GND), D45.5 (GND), D46.5 (GND), D47.5 (GND), D48.5 (GND), D49.5 (GND), D5.5 (GND), D50.5 (GND), D51.5 (GND), D52.5 (GND), D53.5 (GND), D54.5 (GND), D55.5 (GND), D56.5 (GND), D57.5 (GND), D58.5 (GND), D59.5 (GND), D6.5 (GND), D60.5 (GND), D61.5 (GND), D62.5 (GND), D63.5 (GND), D64.5 (GND), D65.5 (GND), D66.5 (GND), D67.5 (GND), D68.5 (GND), D69.5 (GND), D7.5 (GND), D70.5 (GND), D71.5 (GND), D72.5 (GND), D73.5 (GND), D74.5 (GND), D75.5 (GND), D76.5 (GND), D77.5 (GND), D78.5 (GND), D79.5 (GND), D8.5 (GND), D80.5 (GND), D81.5 (GND), D82.5 (GND), D83.5 (GND), D84.5 (GND), D85.5 (GND), D86.5 (GND), D87.5 (GND), D88.5 (GND), D89.5 (GND), D9.5 (GND), D90.5 (GND), D91.5 (GND), D92.5 (GND), D93.5 (GND), D94.5 (GND), D95.5 (GND), D96.5 (GND), D97.5 (GND), D98.5 (GND), D99.5 (GND), H1.1, H2.1, H3.1, H4.1, J3.1 (Pin_1), J4.1 (Pin_1), C?.2, C?.2, C?.2, C?.2, C?.2, C?.2, C?.2, C?.2, C?.2, C?.2, C?.2, C?.2, C?.2, C?.2, C?.2, C?.2, C?.2, C?.2, C?.2, C?.2, C?.2, C?.2, C?.2, C?.2, C?.2, C?.2, C?.2, C?.2, C?.2, C?.2, C?.2, C?.2, C?.2, C?.2, C?.2, C?.2, C?.2, C?.2, C?.2, C?.2, C?.2, C?.2, C?.2, C?.2, C?.2, C?.2, C?.2, C?.2, C?.2, C?.2, C?.2, C?.2, C?.2, C?.2, C?.2, C?.2, C?.2, C?.2, C?.2, C?.2, C?.2, C?.2, C?.2, C?.2, C?.2, C?.2, C?.2, C?.2, C?.2, C?.2, C?.2, C?.2, C?.2, C?.2, C?.2, C?.2, C?.2, C?.2, C?.2, C?.2, C?.2, C?.2, C?.2, C?.2, C?.2, C?.2, C?.2, C?.2, C?.2, C?.2, C?.2, C?.2, C?.2, C?.2, C?.2, C?.2, C?.2, C?.2, C?.2, C?.2, C?.2, C?.2, C?.2, C?.2, C?.2, C?.2, C?.2, C?.2, C?.2, C?.2, C?.2, C?.2, C?.2, C?.2, C?.2, C?.2, C?.2, C?.2, C?.2, C?.2, C?.2, C?.2, C?.2, C?.2, C?.2, C?.2, C?.2, C?.2, C?.2, C?.2, C?.2, C?.2, C?.2, C?.2, C?.2, C?.2, C?.2, C?.2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
- net LED_RXD: now also J3.3 (Pin_3); no longer J3.2 (Pin_2)
- net LED_TXD: now also J3.2 (Pin_2); no longer J3.1 (Pin_1)
- net SCL: now also J4.3 (Pin_3); no longer J4.2 (Pin_2)
- net SDA: now also J4.2 (Pin_2); no longer J4.1 (Pin_1)
Other:
- moved on the sheet: H1, H2, H3, H4, J1, J2, R259
